File: hardware/CH592/OpenDongle-CH592.kicad_pcb (KiCad board)
At the start: 2 copper layers, 16.3 x 9.9 mm, 9 parts, among them J1 PCB USB, U2 XC6206P332MR-G, U3 CH592D, Y1 Crystal

Commit message: fix: Fix library, license and versions
Parts:
- Y1: value Crystal -> 32MHz
Changed lines of the file:
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@@
 			)
 		)
-		(property "Value" "Crystal"
+		(property "Value" "32MHz"
 			(at 0 2.45 0)
 			(layer "F.Fab")
@@
 			)
 		)
+		(attr exclude_from_pos_files exclude_from_bom)
 		(net_tie_pad_groups "1, 2")
 		(duplicate_pad_numbers_are_jumpers no)
@@
 			)
 		)
+		(attr exclude_from_pos_files exclude_from_bom)
 		(duplicate_pad_numbers_are_jumpers no)
 		(fp_line
