File: hardware/CH592/OpenDongle-CH592.kicad_sch (KiCad schematic)
At the start: 9 parts, among them J1 PCB USB, U2 XC6206P332MR-G, U3 CH592D, Y1 Crystal

Commit message: fix: Fix library, license and versions
Parts:
- Y1: value Crystal -> 32MHz
Changed lines of the file:
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@@
 	(title_block
 		(title "OpenDongle CH592")
-		(date "2026-06-07")
-		(rev "0.001")
+		(date "2026-07-12")
+		(rev "0.93")
 		(company "Copyright 2026 Eric Molitor (EMulator)")
-		(comment 3 "github.com/emolitor/ OpenDongle")
-		(comment 4 "CERN-OHL-S CERN Open Hardware Licence Version 2 - Strong-Reciprocal")
+		(comment 3 "github.com/openkeyboard-org/OpenDongle")
+		(comment 4 "CERN-OHL-W CERN Open Hardware Licence Version 2 - Weakly Reciprocal")
 	)
 	(junction
@@
 			)
 		)
-		(property "Value" "Crystal"
+		(property "Value" "32MHz"
 			(at 130.81 109.22 0)
 			(show_name no)
